Commit message: change model to XArm7

File: assets/robot/xarm6_description/xarm7_allegro.urdf (robot description, URDF)
Before this commit: robot xarm6, 31 links, 30 joints
Links:
- removed link world
- added link link7, mass 0.31468; collision mesh filename=meshes/xarm7/collision/link7_vhacd.obj; visual mesh filename=meshes/xarm7/visual/link7_smooth.STL
- link link1: mass 2.16 -> 0.42603; geometry collision mesh filename=meshes/xarm7/collision/link1_vhacd.obj; visual mesh filename=meshes/xarm7/visual/link1_smooth.STL
- link link2: mass 1.71 -> 0.56095; geometry collision mesh filename=meshes/xarm7/collision/link2_vhacd.obj; visual mesh filename=meshes/xarm7/visual/link2_smooth.STL
- link link3: mass 1.384 -> 0.44463; geometry collision mesh filename=meshes/xarm7/collision/link3_vhacd.obj; visual mesh filename=meshes/xarm7/visual/link3_smooth.STL
- link link4: mass 1.115 -> 0.52387; geometry collision mesh filename=meshes/xarm7/collision/link4_vhacd.obj; visual mesh filename=meshes/xarm7/visual/link4_smooth.STL
- link link5: mass 1.275 -> 0.18554; geometry collision mesh filename=meshes/xarm7/collision/link5_vhacd.obj; visual mesh filename=meshes/xarm7/visual/link5_smooth.STL
- link link6: mass 0.1096 -> 0.31344; geometry collision mesh filename=meshes/xarm7/collision/link6_vhacd.obj; visual mesh filename=meshes/xarm7/visual/link6_smooth.STL
- link link_base: mass 2.7 -> 0.88556; geometry collision mesh filename=meshes/xarm7/collision/linkbase.obj; visual mesh filename=meshes/xarm7/visual/link_base_smooth.STL
Joints:
- removed joint world_joint
- added joint joint7: type revolute, parent link6, child link7, origin xyz=0.076 0.097 0 rpy=-1.5708 0 0, axis 0 0 1, limit lower=-6.28318530718 upper=6.28318530718 effort=20 velocity=3.14
- joint gripper_base_joint: parent link6 -> link7
- joint joint1: limit lower=-6.28318530718 upper=6.28318530718 effort=50.0 velocity=3.14 -> lower=-6.28318530718 upper=6.28318530718 effort=50 velocity=3.14
- joint joint2: limit lower=-2.059 upper=2.0944 effort=50.0 velocity=3.14 -> lower=-2.059 upper=2.0944 effort=50 velocity=3.14
- joint joint3: limit lower=-3.927 upper=0.19198 effort=32.0 velocity=3.14 -> lower=-6.28318530718 upper=6.28318530718 effort=30 velocity=3.14; origin xyz=0.0535 -0.2845 0 rpy=0 0 0 -> xyz=0 -0.293 0 rpy=1.5708 0 0
- joint joint4: limit lower=-6.28318530718 upper=6.28318530718 effort=32.0 velocity=3.14 -> lower=-0.19198 upper=3.927 effort=30 velocity=3.14; origin xyz=0.0775 0.3425 0 rpy=-1.5708 0 0 -> xyz=0.0525 0 0 rpy=1.5708 0 0
- joint joint5: limit lower=-1.69297 upper=3.14159265359 effort=32.0 velocity=3.14 -> lower=-6.28318530718 upper=6.28318530718 effort=30 velocity=3.14; origin xyz=0 0 0 rpy=1.5708 0 0 -> xyz=0.0775 -0.3425 0 rpy=1.5708 0 0
- joint joint6: limit lower=-6.28318530718 upper=6.28318530718 effort=20.0 velocity=3.14 -> lower=-1.69297 upper=3.14159265359 effort=20 velocity=3.14; origin xyz=0.076 0.097 0 rpy=-1.5708 0 0 -> xyz=0 0 0 rpy=1.5708 0 0
